File: Hardware/SendoXBati/Sendo_X_Bati/Sendo_X_Bati.kicad_sch (KiCad schematic)
At the start: 35 parts, among them J1 TB_1X2, J2 Ultrasonido, J3 Ultrasonido, J4 CNY70, J5 CNY70, J6 TB_1X2, J7 TB_1X2, J8 Conn_01x04, SW1 SW_SPDT, SW2 SW_Push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

Commit message: actualizacion del sch de placa sendoXbati
Parts:
- removed C10, C7, C8, C9: C, symbol Device:C
- removed J2, J3: Ultrasonido, Connector_JST:JST_EH_B4B-EH-A_1x04_P2.50mm_Vertical, symbol EESTN5:Conn_01x04
- removed U4, U5: TB67H450FNG_EL, P-HSOP8-0405-1p27-002_TOS, symbol 2023-08-25_03-42-01:TB67H450FNG_EL
- added D2: LED, symbol Device:LED
- added J10, J11, J12, J13, J2: sharp1, symbol EESTN5:CONN_01X03
- added J14: Ultrasonido, Connector_JST:JST_EH_B4B-EH-A_1x04_P2.50mm_Vertical, symbol EESTN5:Conn_01x04
- added J3: sensor2, symbol EESTN5:CONN_01X03
- added J9: potencia, symbol EESTN5:TB_1X2
- added JP1: Jumper, symbol EESTN5:Jumper
- added R6: R, symbol Device:R
- J1: value TB_1X2 -> logica
- J4, J5: value CNY70 -> sharp1; footprint Connector_JST:JST_PH_B3B-PH-K_1x03_P2.00mm_Vertical -> (none)
- U3: value LM2596S-3.3 -> LM2596S
Connections:
- net CNY70_FD is gone; now on net +5V: J4.1 (P1)
- net CNY70_FI is gone; now on net +5V: J5.1 (P1)
- net RX is gone; now on net RXD: J8.2 (Pin_2)
- net TX is gone; now on net TXD: J8.1 (Pin_1)
- net +5V: now also J10.1 (P1), J11.1 (P1), J12.1 (P1), J13.1 (P1), J14.2 (Pin_2), J2.1 (P1), J3.1 (P1), R6.2; no longer J4.2 (P2), J5.2 (P2)
- net +BATT: now also JP1.2 (B); no longer C4.1, C5.1, SW1.1 (A), U3.1 (VIN)
- net AIN1: now also U1.18 (NC@18)
- net AIN2: now also U1.19 (NC@19)
- net BIN1: now also U1.28 (IO17)
- net BIN2: now also U1.27 (IO16)
- net Echo_1: now also J14.4 (Pin_4)
- net GND: now also J4.2 (P2), J5.2 (P2), D2.1 (K), J10.2 (P2), J11.2 (P2), J12.2 (P2), J13.2 (P2), J14.1 (Pin_1), J2.2 (P2), J3.2 (P2), J9.2; no longer J4.3 (P3), J5.3 (P3)
- net SCL: now also U1.36 (IO22)
- net SDA: now also U1.33 (IO21)
- net Trigger_1: now also J14.3 (Pin_3)
- net sensor4: now reaches U1.10 (IO25)
- net sensor4: now also J11.3 (P3)
- net echo_1: now reaches U1.11 (IO26)
- net trigger_1: now reaches U1.12 (IO27)
- net sensor8: now reaches U1.30 (IO18)
- net sensor8: now also J13.3 (P3)
- net sensor7: now reaches U1.31 (IO19)
- net sensor7: now also J5.3 (P3)
- net sensor6: now reaches U1.32 (NC@32)
- net sensor6: now also J12.3 (P3)
- net RXD: now reaches U1.34 (IO3)
- net TXD: now reaches U1.35 (IO1)
- net start: now reaches U1.37 (IO23)
- net start: now also R4.2, SW3.1
- net sensor1: now reaches U1.6 (IO34)
- net sensor1: now also J2.3 (P3)
- net sensor2: now reaches U1.7 (IO35)
- net sensor2: now also J3.3 (P3)
- net sensor3: now reaches U1.8 (IO32)
- net sensor3: now also J10.3 (P3)
- net sensor5: now reaches U1.9 (IO33)
- net sensor5: now also J4.3 (P3)
- new net: D2.2 (A), R6.1
- new net: J9.1, JP1.1 (A)
- new net +7.5V: C4.1, C5.1, SW1.1 (A), U3.1 (VIN)
- no-connect marks 0 -> 4
Other:
- added sheet drivers (driver motor.kicad_sch)
- note added: "driver motor"
- note removed: "DRIVERS"
- note removed: "SENSORES CNY70 (PISO)"
- moved on the sheet: J1, SW1
